Commit message: add SensOne model in urdf and srdf

File: dual_arm_panda_ur_moveit_config/config/ur_macro.xacro (robot description, xacro)
@@ -410,9 +410,37 @@
       <child link="${prefix}tool0"/>
     </joint>
+    <joint name="${prefix}ur_to_sensone_joint" type="fixed">
+      <parent link="${prefix}tool0" />
+      <child link="${prefix}sensone_link" />
+      <origin xyz="0 0 0.036" rpy="0 0 0" />
+    </joint>
+    <link name="${prefix}sensone_link">
+      <visual>
+        <origin xyz="0 0 0" rpy="0 0 0" />
+        <geometry>
+          <mesh
+            filename="package://robotiq_description/meshes/visual/2f_85/SensONE_scaled.dae" />
+        </geometry>
+      </visual>
+      <collision>
+        <origin xyz="0 0 0" rpy="0 0 0" />
+        <geometry>
+          <mesh
+            filename="package://robotiq_description/meshes/collision/2f_85/SensONE_scaled.stl" />
+        </geometry>
+      </collision>
+      <inertial>
+        <mass value="0.01" />
+        <origin xyz="0 0 0" />
+        <inertia ixx="0.000044" ixy="0.0" ixz="0.0" iyy="0.000027" iyz="0.0" izz="0.000027" />
+      </inertial>
+    </link>
     <joint name="${prefix}ur_to_robotiq_joint" type="fixed">
       <!-- The parent link must be read from the robot model it is attached to. -->
-      <parent link="${prefix}tool0" />
+      <parent link="${prefix}sensone_link" />
+      <!-- <parent link="${prefix}tool0" /> -->
       <child link="${prefix}ur_to_robotiq_link" />
       <origin xyz="0 0 0" rpy="0 0 0" />
+      <!-- <origin xyz="0 0 0" rpy="0 0 0" /> -->
     </joint>
     <link name="${prefix}ur_to_robotiq_link">
